File: pcb/pcb.kicad_pcb (KiCad board)
At the start: 2 copper layers, 139.8 x 110.8 mm, 114 parts, among them SW1 Switch, SW10 Switch, SW11 Switch, SW12 Switch, SW13 Switch, SW14 Switch, SW15 Switch, SW16 Switch, SW17 Switch, SW18 Switch, SW19 Switch, SW2 Switch, SW20 Switch, SW21 Switch, SW22 Switch, SW23 Switch, SW24 Switch, SW25 Switch, SW26 Switch, SW27 Switch, SW28 Switch, SW29 Switch, SW3 Switch, SW30 Switch, SW31 Switch, SW32 Switch, SW33 Switch, SW34 Switch, SW4 Switch, SW5 Switch, SW6 Switch, SW7 Switch, SW8 Switch, SW9 Switch

Commit message: pcb updates
Parts:
- moved D33 9.22 mm to (119.5, 166.5)
- moved REF** 0.50 mm to (147.0, 71.0)
Routing:
- net VCC: track 808.4 -> 845.8 mm
- net row3: track 197.0 -> 210.6 mm
- net Net-(D33-A): track 6.86 -> 13.5 mm
- net Net-(LED27-DOUT): track 36.5 -> 34.4 mm
- net row4: track 247.2 -> 248.7 mm
- net Net-(LED28-DOUT): track 17.0 -> 17.7 mm
- net row0: track 218.7 -> 218.1 mm
Other:
- board text added: "KeyGameBoard v1.0"
- board text removed: "v1.0"

Commit message: PCB 1.1
Parts:
- moved LED17 0.20 mm to (106.0, 93.3)
- moved LED21 0.20 mm to (125.0, 114.3)
- moved LED20 0.20 mm to (125.0, 133.3)
- moved LED28 0.10 mm to (146.1, 159.5)
Connections:
- LED1 pad 3: unconnected-(LED1-VSS-Pad3) -> GND
- LED2 pad 3: unconnected-(LED2-VSS-Pad3) -> GND
- LED3 pad 3: unconnected-(LED3-VSS-Pad3) -> GND
Routing:
- net GND: vias 3 -> 4
Other:
- board text added: "KeyGameBoard v1.1"
- board text removed: "KeyGameBoard v1.0"
