File: pcb/pcb.kicad_sch (KiCad schematic)
At the start: 113 parts, among them SW1 Switch, SW10 Switch, SW11 Switch, SW12 Switch, SW13 Switch, SW14 Switch, SW15 Switch, SW16 Switch, SW17 Switch, SW18 Switch, SW19 Switch, SW2 Switch, SW20 Switch, SW21 Switch, SW22 Switch, SW23 Switch, SW24 Switch, SW25 Switch, SW26 Switch, SW27 Switch, SW28 Switch, SW29 Switch, SW3 Switch, SW30 Switch, SW31 Switch, SW32 Switch, SW33 Switch, SW34 Switch, SW4 Switch, SW5 Switch, SW6 Switch, SW7 Switch, SW8 Switch, SW9 Switch

Commit message: PCB 1.1
Connections:
- net GND: now also LED1.3 (VSS), LED2.3 (VSS), LED3.3 (VSS)
Changed lines of the file:
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@@
   (junction (at 198.12 119.38) (diameter 0) (color 0 0 0 0)
   )
+  (junction (at 182.88 119.38) (diameter 0) (color 0 0 0 0)
+  )
   (junction (at 87.63 162.56) (diameter 0) (color 0 0 0 0)
   )
@@
   (junction (at 34.29 121.92) (diameter 0) (color 0 0 0 0)
   )
+  (junction (at 182.88 134.62) (diameter 0) (color 0 0 0 0)
+  )
   (junction (at 322.58 134.62) (diameter 0) (color 0 0 0 0)
   )
@@
   )
   (junction (at 274.32 104.14) (diameter 0) (color 0 0 0 0)
+  )
+  (junction (at 209.55 144.78) (diameter 0) (color 0 0 0 0)
   )
   (junction (at 105.41 142.24) (diameter 0) (color 0 0 0 0)
@@
     (stroke (width 0) (type default))
   )
+  (wire (pts (xy 182.88 104.14) (xy 182.88 119.38))
+    (stroke (width 0) (type default))
+  )
   (wire (pts (xy 85.09 113.03) (xy 85.09 133.35))
     (stroke (width 0) (type default))
@@
     (stroke (width 0) (type default))
   )
+  (wire (pts (xy 182.88 134.62) (xy 182.88 144.78))
+    (stroke (width 0) (type default))
+  )
   (wire (pts (xy 36.83 35.56) (xy 39.37 35.56))
     (stroke (width 0) (type default))
@@
     (stroke (width 0) (type default))
   )
+  (wire (pts (xy 182.88 119.38) (xy 182.88 134.62))
+    (stroke (width 0) (type default))
+  )
   (wire (pts (xy 295.91 104.14) (xy 295.91 88.9))
     (stroke (width 0) (type default))
@@
     (stroke (width 0) (type default))
   )
+  (wire (pts (xy 182.88 144.78) (xy 209.55 144.78))
+    (stroke (width 0) (type default))
+  )
